File: keypad.sch (KiCad schematic (older format))
At the start: 27 parts

Commit message: footprints
footprints done
Parts:
- C1, C2, C3, C4, C5, C6, C7: renamed from C?; footprint (none) -> Capacitor_SMD:C_0805_2012Metric
- D1, D2, D3, D4, D5, D6: renamed from D?; footprint (none) -> Diode_SMD:D_SOD-123
- F1: renamed from F?; footprint (none) -> Fuse:Fuse_1206_3216Metric
- MX1, MX2, MX3, MX4, MX5, MX6: renamed from MX?; footprint (none) -> MX_Only:MXOnly-1U-Hotswap
- R1, R2, R3: renamed from R?; footprint (none) -> Resistor_SMD:R_0805_2012Metric
- SW1: renamed from SW?; footprint (none) -> random-keyboard-parts:SKQG-1155865
- USB1: renamed from USB?; footprint (none) -> random-keyboard-parts:Molex-0548190589
- Y1: renamed from Y?; footprint (none) -> Crystal:Crystal_SMD_3225-4Pin_3.2x2.5mm
- gave numbers to parts that had none: 1
