File: keypad.kicad_pcb (KiCad board)
At the start: 2 copper layers, 27 parts, among them SW1 SW_Push, U1 ATmega32U4-AU, Y1 16MHz

Commit message: routing
first routing
Parts:
- C3, C4, C5, C6, C7, F1, R1, R2, R3, SW1, USB1: moved to B.Cu
- moved C6 51.2 mm to (165.1, 127.5)
- moved R1 47.6 mm to (163.3, 115.3), turned to 90 degrees
- moved R3 43.3 mm to (194.9, 127.4), turned to 90 degrees
- moved SW1 38.5 mm to (162.1, 135.4), turned to 180 degrees
- moved R2 35.3 mm to (166.0, 115.3), turned to 90 degrees
- moved C7 26.1 mm to (173.1, 115.5), turned to 90 degrees
- moved C3 26.0 mm to (195.2, 116.0), turned to 90 degrees
- moved C5 24.5 mm to (190.9, 131.8), turned to 180 degrees
- moved USB1 20.8 mm to (165.1, 104.1), turned to 270 degrees
- moved C4 19.7 mm to (181.2, 131.8)
- moved C1 16.9 mm to (181.5, 111.7), turned to 90 degrees
- moved Y1 16.7 mm to (186.0, 111.8), turned to 270 degrees
- moved F1 9.16 mm to (159.9, 116.8), turned to 90 degrees
- moved C2 2.12 mm to (190.2, 111.7), turned to 270 degrees
Routing:
- net GND: track 0.00 -> 130.9 mm, vias 0 -> 3
- net +5V: track 0.00 -> 97.4 mm, vias 0 -> 4
- net ROW1: track 0.00 -> 77.2 mm
- net COL2: track 0.00 -> 70.6 mm, vias 0 -> 4
- net ROW0: track 0.00 -> 68.7 mm
- net COL1: track 0.00 -> 50.4 mm, vias 0 -> 2
- net Net-(SW1-Pad2): track 0.00 -> 35.4 mm, vias 0 -> 2
- net COL0: track 0.00 -> 26.6 mm, vias 0 -> 2
- net Net-(R1-Pad1): track 0.00 -> 22.6 mm
- net Net-(R2-Pad1): track 0.00 -> 21.2 mm
- net Net-(C2-Pad1): track 0.00 -> 12.3 mm
- net Net-(C7-Pad1): track 0.00 -> 9.58 mm
- net VCC: track 0.00 -> 9.23 mm
- net Net-(C1-Pad1): track 0.00 -> 7.72 mm
- net D-: track 0.00 -> 6.17 mm
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Other:
- board outline added: 101.6 x 38.1 mm
- net class Default: trace_width 0.25 -> 0.254
- net class Power added: clearance 0.2, trace_width 0.381, via_dia 0.8, via_drill 0.4

Commit message: routing/fill
complte
Parts:
- moved USB1 0.14 mm to (165.0, 104.1)
Routing:
- net GND: track 130.9 -> 97.1 mm, vias 3 -> 0
- net +5V: track 97.4 -> 112.0 mm, vias 4 -> 6
- added copper zone on B.Cu, net GND
Changed lines of the file:
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@@
     (thickness 1.6)
     (drawings 8)
-    (tracks 245)
+    (tracks 243)
     (zones 0)
     (modules 27)
@@
   )
   (module random-keyboard-parts:Molex-0548190589 (layer B.Cu)
-    (at 165.133 104.085 270)
+    (at 165.006 104.14 270)
     (attr smd)
     (fp_text reference USB1 (at 2.032 0 180) (layer B.SilkS)
@@
   (segment (start 188.747 131.1685) (end 188.747 129.946) (width 0.381) (layer B.Cu) (net 1))
   (segment (start 188.747 129.946) (end 188.747 129.259) (width 0.381) (layer B.Cu) (net 1))
-  (via (at 167.64 127.508) (size 0.8) (drill 0.4) (layers F.Cu B.Cu) (net 1))
   (segment (start 166.0375 127.4595) (end 167.5915 127.4595) (width 0.381) (layer B.Cu) (net 1))
   (segment (start 167.5915 127.4595) (end 167.64 127.508) (width 0.381) (layer B.Cu) (net 1))
-  (via (at 170.307 116.332) (size 0.8) (drill 0.4) (layers F.Cu B.Cu) (net 1))
-  (segment (start 167.64 127.508) (end 170.307 124.841) (width 0.381) (layer F.Cu) (net 1))
-  (segment (start 170.307 124.841) (end 170.307 116.332) (width 0.381) (layer F.Cu) (net 1))
   (segment (start 170.307 113.157) (end 170.3685 113.0955) (width 0.381) (layer B.Cu) (net 1))
   (segment (start 170.307 116.332) (end 170.307 113.157) (width 0.381) (layer B.Cu) (net 1))
   (segment (start 166.733 109.46) (end 170.3685 113.0955) (width 0.381) (layer B.Cu) (net 1))
   (segment (start 170.3685 113.0955) (end 171.827 114.554) (width 0.381) (layer B.Cu) (net 1))
-  (segment (start 167.64 127.508) (end 167.64 128.073685) (width 0.381) (layer F.Cu) (net 1))
-  (segment (start 167.64 128.073685) (end 167.64 138.176) (width 0.381) (layer F.Cu) (net 1))
-  (segment (start 167.64 138.176) (end 166.751 139.065) (width 0.381) (layer F.Cu) (net 1))
-  (via (at 157.099 139.065) (size 0.8) (drill 0.4) (layers F.Cu B.Cu) (net 1))
-  (segment (start 166.751 139.065) (end 157.099 139.065) (width 0.381) (layer F.Cu) (net 1))
   (segment (start 157.099 139.065) (end 157.099 137.414) (width 0.381) (layer B.Cu) (net 1))
   (segment (start 157.226 137.287) (end 159.004 137.287) (width 0.381) (layer B.Cu) (net 1))
@@
   (segment (start 191.867 131.826) (end 191.867 129.792) (width 0.381) (layer B.Cu) (net 4))
   (segment (start 191.867 129.792) (end 190.203 128.128) (width 0.381) (layer B.Cu) (net 4))
+  (via (at 191.262 133.477) (size 0.8) (drill 0.4) (layers F.Cu B.Cu) (net 4))
+  (segment (start 191.867 131.826) (end 191.867 132.872) (width 0.381) (layer B.Cu) (net 4))
+  (segment (start 191.867 132.872) (end 191.262 133.477) (width 0.381) (layer B.Cu) (net 4))
+  (via (at 180.213 133.477) (size 0.8) (drill 0.4) (layers F.Cu B.Cu) (net 4))
+  (segment (start 191.262 133.477) (end 180.213 133.477) (width 0.381) (layer F.Cu) (net 4))
+  (segment (start 180.213 131.856) (end 180.243 131.826) (width 0.381) (layer B.Cu) (net 4))
+  (segment (start 180.213 133.477) (end 180.213 131.856) (width 0.381) (layer B.Cu) (net 4))
   (segment (start 178.843 122.428) (end 179.847 122.428) (width 0.254) (layer B.Cu) (net 5))
   (segment (start 178.5125 122.428) (end 178.843 122.428) (width 0.254) (layer B.Cu) (net 5))
@@
   (segment (start 181.939 115.316) (end 182.347 115.724) (width 0.254) (layer B.Cu) (net 23))
   (segment (start 177.673 115.316) (end 181.939 115.316) (width 0.254) (layer B.Cu) (net 23))
+  (zone (net 1) (net_name GND) (layer B.Cu) (hatch edge 0.508)
+    (connect_pads (clearance 0.508))
+    (min_thickness 0.254)
+    (fill yes (arc_segments 32) (thermal_gap 0.508) (thermal_bridge_width 0.508))
+    (polygon
+      (pts
+        (xy 154.813 102.362) (xy 197.485 102.362) (xy 197.612 140.462) (xy 154.813 140.462)
+      )
+    )
+  )
 )
