File: pcb/keypad.kicad_pcb (KiCad board)
At the start: 2 copper layers, 99.2 x 38.1 mm, 27 parts, among them SW1 SW_Push, U1 ATmega32U4-AU, Y1 16MHz

Commit message: a
a
Parts:
- moved F1 7.64 mm to (166.7, 122.4)
- moved C6 5.56 mm to (170.5, 126.2)
- moved USB1 4.29 mm to (172.6, 104.2)
- moved SW1 4.29 mm to (174.7, 137.1)
Routing:
- net +5V: track 111.4 -> 102.2 mm
- net VCC: track 9.59 -> 18.3 mm
- net D-: track 5.99 -> 10.2 mm
- net D+: track 5.95 -> 8.98 mm
- net GND: track 84.2 -> 82.7 mm
- net Net-(SW1-Pad2): track 26.9 -> 28.3 mm
Other:
- outline, holes or cut-outs redrawn
