File: pcb/keypad.kicad_pcb (KiCad board)
At the start: 2 copper layers, 99.2 x 38.1 mm, 27 parts, among them SW1 SW_Push, U1 ATmega32U4-AU, Y1 16MHz

Commit message: cad, pcb fixes
a
Parts:
- moved SW1 10.3 mm to (184.2, 141.0)
- moved USB1 8.54 mm to (178.3, 97.9)
Routing:
- net Net-(SW1-Pad2): track 28.3 -> 40.1 mm
- net VCC: track 18.3 -> 28.8 mm
- net D-: track 10.2 -> 19.1 mm
- net D+: track 8.98 -> 17.7 mm
- net GND: track 82.7 -> 88.3 mm
Other:
- board size 99.2 x 38.1 mm -> 99.2 x 50.8 mm
